File: hardware/rev2/JardinIOT/ESP32.brd (EAGLE design)
At the start: 160 x 100 mm, 5 parts, among them IC1 7815TV

Commit message: WIP: Sync au repo personnel de Vincent (#87)
Parts:
- added C3: 0.33µF, rcl:C0805
- added C4: 0.1µF, rcl:C0805
- added IC2: 7812TV, linear:TO220V
- added Q1, Q2, Q3, Q4: BD243, transistor-npn:TO220
- added R1, R2: 220Ω, rcl:0204/5
- added R10, R4, R6, R8: 24 OHM, rcl:0204/7
- added R3, R5, R7, R9: 12 OHM, rcl:0204/7
- added S1, S2: (no value), switch-omron:B3F-10XX
- added X2, X3, X4, X6: (no value), con-wago-500:W237-102
- added X5, X7, X8, X9: (no value), con-wago-500:W237-103
- IC1: value 7815TV -> 7805TV
- X1: device con-wago-500:W237-113 -> con-wago-500:W237-102
- moved X1 101.6 mm to (111.8, 92.7)
- moved U$1 35.1 mm to (61.0, 52.1), turned to 180 degrees
- moved IC1 29.2 mm to (11.4, 50.8)
- moved C2 26.9 mm to (10.2, 47.0), turned to 0 degrees
- moved C1 11.4 mm to (12.7, 62.2), turned to 180 degrees
Connections:
- removed net 20V_VCC: C1.1, IC1.1, X1.1
- new net 12V_VCC: C4.1, IC2.3, R3.2, R5.2, R7.2, R9.2
- new net 20VDC: C1.1, C3.1, IC1.1, IC2.1, X6.1
- new net 3V3: R1.2, R2.2, U$1.1, X5.3, X7.3, X8.3, X9.3
- new net N$1: R1.1, S1.1, S1.2, U$1.4
- new net N$10: Q3.2, R7.1
- new net N$11: Q3.1, R8.1
- new net N$12: Q4.3, X4.2
- new net N$13: Q4.2, R9.1
- new net N$14: Q4.1, R10.1
- new net N$15: R4.2, U$1.7
- new net N$16: U$1.22, X5.2
- new net N$17: R8.2, U$1.6
- new net N$18: R6.2, U$1.8
- new net N$19: R10.2, U$1.5
- new net N$20: U$1.21, X7.2
- new net N$21: U$1.20, X8.2
- new net N$22: U$1.19, X9.2
- new net N$3: R2.1, S2.1, S2.2, U$1.3
- new net N$4: Q1.2, R3.1
- new net N$5: Q1.1, R4.1
- new net N$6: Q2.3, X1.2
- new net N$7: Q2.2, R5.1
- new net N$8: Q2.1, R6.1
- new net N$9: Q3.3, X3.2
- net GND: now also C3.2, C4.2, IC2.2, S1.3, S1.4, S2.3, S2.4, X1.1, X2.1, X3.1, X4.1, X5.1, X6.2, X7.1, X8.1, X9.1; no longer X1.2
- net N$2: now also Q1.3, X2.2; no longer U$1.1
Routing:
- net GND: track 78.9 -> 585.4 mm
- net 3V3: track 0.00 -> 288.1 mm
- net 12V_VCC: track 0.00 -> 242.2 mm
- net N$19: track 0.00 -> 122.8 mm
- net N$17: track 0.00 -> 110.7 mm
- net N$15: track 0.00 -> 99.2 mm
- net N$1: track 0.00 -> 95.3 mm
- net N$3: track 0.00 -> 91.7 mm
- net N$18: track 0.00 -> 90.0 mm
- net 20VDC: track 0.00 -> 72.2 mm
- net N$16: track 0.00 -> 65.7 mm
- net 5V_VCC: track 45.9 -> 108.9 mm
- net N$20: track 0.00 -> 50.7 mm
- net N$2: track 0.00 -> 45.6 mm
- net N$9: track 0.00 -> 45.6 mm
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Other:
- board text added: "ACTIONNEURS"
- board text added: "CAPTEURS"
- board text added: "Club CEDILLE: https://cedille.etsmtl.ca/"
- board text added: "VIN"
- board text removed: "20/03/2020"
