File: hardware/rev2/JardinIOT/ESP32.sch (EAGLE design)
At the start: 5 parts, among them IC1 7815TV

Commit message: WIP: Sync au repo personnel de Vincent (#87)
Parts:
- added C3: 0.33µF, rcl:C-USC0805
- added C4: 0.1µF, rcl:C-USC0805
- added IC2: 7812TV, linear:7812TV
- added Q1, Q2, Q3, Q4: BD243, transistor-npn:BD243
- added R1, R2: 220Ω, rcl:R-US_0204/5
- added R10, R4, R6, R8: 24 OHM, rcl:R-US_0204/7
- added R3, R5, R7, R9: 12 OHM, rcl:R-US_0204/7
- added S1, S2: (no value), switch-omron:10-XX
- added X2, X3, X4, X6: (no value), con-wago-500:W237-102
- added X5, X7, X8, X9: (no value), con-wago-500:W237-103
- IC1: value 7815TV -> 7805TV; device linear:7815TV -> linear:7805TV
- X1: device con-wago-500:W237-113 -> con-wago-500:W237-102
Connections:
- removed net 20V_VCC: C1.1, IC1.VI, X1-1.KL
- new net 12V_VCC: C4.1, IC2.VO, R3.2, R5.2, R7.2, R9.2
- new net 20VDC: C1.1, C3.1, IC1.VI, IC2.VI, X6-1.KL
- new net 3V3: R1.2, R2.2, U$1.3V3, X5-3.KL, X7-3.KL, X8-3.KL, X9-3.KL
- new net N$1: R1.1, S1.S, S1.S1, U$1.IO2
- new net N$10: Q3.C, R7.1
- new net N$11: Q3.B, R8.1
- new net N$12: Q4.E, X4-2.KL
- new net N$13: Q4.C, R9.1
- new net N$14: Q4.B, R10.1
- new net N$15: R4.2, U$1.IO17
- new net N$16: U$1.IO33, X5-2.KL
- new net N$17: R8.2, U$1.IO16
- new net N$18: R6.2, U$1.IO5
- new net N$19: R10.2, U$1.IO4
- new net N$20: U$1.IO32, X7-2.KL
- new net N$21: U$1.IO35, X8-2.KL
- new net N$22: U$1.IO34, X9-2.KL
- new net N$3: R2.1, S2.S, S2.S1, U$1.IO15
- new net N$4: Q1.C, R3.1
- new net N$5: Q1.B, R4.1
- new net N$6: Q2.E, X1-2.KL
- new net N$7: Q2.C, R5.1
- new net N$8: Q2.B, R6.1
- new net N$9: Q3.E, X3-2.KL
- net GND: now also C3.2, C4.2, IC2.GND, S1.P, S1.P1, S2.P, S2.P1, X1-1.KL, X2-1.KL, X3-1.KL, X4-1.KL, X5-1.KL, X6-2.KL, X7-1.KL, X8-1.KL, X9-1.KL; no longer X1-2.KL
- net N$2: now also Q1.E, X2-2.KL; no longer U$1.3V3
Other:
- moved on the sheet: C2, X1-1, X1-2
